Commit message: - made a new readme and added new environments

File: qarm_gripper/urdf/qarm_gripper.urdf (robot description, URDF)
Before this commit: robot qarm_gripper, 5 links, 4 joints
Joints:
- joint Joint1A: limit lower=0 upper=0 effort=0 velocity=0 -> lower=0 upper=0.9 effort=5 velocity=1
- joint Joint1B: limit lower=0 upper=0 effort=0 velocity=0 -> lower=0 upper=0.9 effort=5 velocity=1
- joint Joint2A: limit lower=0 upper=0 effort=0 velocity=0 -> lower=0 upper=0.9 effort=5 velocity=1
- joint Joint2B: limit lower=0 upper=0 effort=0 velocity=0 -> lower=0 upper=0.9 effort=5 velocity=1
